File: elec/elec.kicad_pcb (KiCad board)
At the start: 2 copper layers, 120 x 140 mm, 80 parts, among them J1 XT60-M, Q1 AON6354, Q2 AON6354, Q3 AON6354, Q4 AON6354, SW1 SW_SPST, SW2 SW_SPST, U1 TPS5430DDA, U10 XT30UPB-M, U11 VNH5019ATR-E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

Commit message: completed?
Parts:
- removed C11, C12: 470u, Capacitor_THT:CP_Radial_D8.0mm_P3.50mm
- removed Q3, Q4: AON6354, initium20:8-DFN (5x6)
- removed R24, R25, R32, R33: 3K3, Resistor_SMD:R_0603_1608Metric
- removed R26, R34: 10K, Resistor_SMD:R_0603_1608Metric
- removed R27, R28, R29, R30, R31, R35, R36, R37, R38, R39: 1K, Resistor_SMD:R_0603_1608Metric
- removed SW1: SW_SPST, Connector_AMASS:AMASS_XT60-M_1x02_P7.20mm_Vertical
- removed TP1: TestPoint_2Pole, TestPoint:TestPoint_2Pads_Pitch2.54mm_Drill0.8mm
- removed U10, U12: XT30UPB-M, Connector_AMASS:AMASS_XT30UPB-M_1x02_P5.0mm_Vertical
- removed U11: VNH5019ATR-E, initium20:VNH5019ATR-E
- added H1: MountingHole, MountingHole:MountingHole_3.2mm_M3_Pad, F.Cu at (133.5, 67.2)
- added H2: MountingHole, MountingHole:MountingHole_3.2mm_M3_Pad, F.Cu at (263.5, 67.3)
- added H3: MountingHole, MountingHole:MountingHole_3.2mm_M3_Pad, F.Cu at (133.5, 227.3)
- added H4: MountingHole, MountingHole:MountingHole_3.2mm_M3_Pad, F.Cu at (263.5, 227.2)
- R5, R6: value R -> 10K
- U9: value VNH5019ATR-E -> 113991054; footprint initium20:VNH5019ATR-E -> initium20:XiaoSeeedStudioEsp32
- moved U4 196.4 mm to (167.0, 228.8)
- moved R7 142.4 mm to (179.4, 217.6), turned to 180 degrees
- moved SW2 141.7 mm to (178.8, 221.6), turned to 0 degrees
- moved U9 93.3 mm to (198.5, 215.3), turned to 180 degrees
- moved Q1 90.1 mm to (173.1, 166.7), turned to 0 degrees
- moved R8 84.8 mm to (172.8, 173.1), turned to 180 degrees
- moved R14 83.7 mm to (172.8, 174.6), turned to 180 degrees
- moved R12 82.7 mm to (172.8, 176.1), turned to 180 degrees
- moved R10 81.7 mm to (172.8, 177.6), turned to 180 degrees
- moved R15 80.8 mm to (172.8, 179.1), turned to 180 degrees
- moved R11 79.9 mm to (172.8, 180.6), turned to 180 degrees
- moved R13 79.1 mm to (172.8, 182.1), turned to 180 degrees
- moved R9 78.3 mm to (172.8, 183.6), turned to 180 degrees
- moved A1 75.0 mm to (200.6, 177.1)
- moved R5 71.4 mm to (194.7, 141.3)
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Connections:
- A1 pad 10: /Motor 4 IN A -> unconnected-(A1-Pad10)
- A1 pad 11: /Motor 4 IN B -> unconnected-(A1-Pad11)
- A1 pad 2: /Motor 3 PWM -> unconnected-(A1-Pad2)
- A1 pad 20: unconnected-(A1-Pad20) -> /ESP32 RX
- A1 pad 21: unconnected-(A1-Pad21) -> /ESP32 TX
- A1 pad 3: /Motor 4 PWM -> unconnected-(A1-Pad3)
- A1 pad 8: /Motor 3 IN A -> unconnected-(A1-Pad8)
- A1 pad 9: /Motor 3 IN B -> unconnected-(A1-Pad9)
- J1 pad P: Net-(J1-POS) -> +12V
- TP2 pad 2: Net-(J1-POS) -> +12V
- U9 pad 1: /Motor 3/Motor Out A -> unconnected-(U9-D0-Pad1)
- U9 pad 10: Net-(U9-INB) -> unconnected-(U9-D9-Pad10)
- U9 pad 11: Net-(Q3-G) -> unconnected-(U9-D10-Pad11)
- U9 pad 12: +12V -> unconnected-(U9-VCC_3V3-Pad12)
- U9 pad 13: Net-(C11-Pad1) -> GND
- U9 pad 14: (no net) -> +5V
- U9 pad 2: (no net) -> unconnected-(U9-D1-Pad2)
- U9 pad 3: Net-(C11-Pad1) -> unconnected-(U9-D2-Pad3)
- U9 pad 4: Net-(U9-INA) -> unconnected-(U9-D3-Pad4)
- U9 pad 5: Net-(U9-ENA/DIAGA) -> unconnected-(U9-D4-Pad5)
- U9 pad 7: Net-(U9-PWM) -> /ESP32 TX
- U9 pad 8: unconnected-(U9-CS-Pad8) -> /ESP32 RX
- U9 pad 9: Net-(U9-ENB/DIAGB) -> unconnected-(U9-D8-Pad9)
Routing:
- net +5V: track 23.4 -> 399.7 mm, vias 0 -> 3
- net +12V: track 3.83 -> 313.6 mm, vias 1 -> 13
- net +3V3: track 23.7 -> 297.2 mm, vias 0 -> 6
- net /Motors Enable: track 0.00 -> 159.1 mm, vias 0 -> 4
- net /ESP32 TX: track 0.00 -> 66.7 mm
- net /ESP32 RX: track 0.00 -> 55.2 mm, vias 0 -> 1
- net /Motor 2 PWM: track 0.00 -> 51.3 mm
- net /Motor 2 IN A: track 1.50 -> 42.2 mm
- net /Motor 1 IN B: track 1.50 -> 34.8 mm
- net /Motor 2 IN B: track 1.50 -> 30.0 mm, vias 0 -> 1
- net /Motor 1 IN A: track 1.50 -> 26.5 mm, vias 0 -> 1
- net /RX (IMU): track 4.02 -> 25.4 mm
- net /Motor 1 PWM: track 0.00 -> 18.6 mm
- net /TX (IMU): track 4.02 -> 21.6 mm, vias 0 -> 1
- net Net-(Q3-G): track 7.17 -> 0.00 mm, vias 2 -> 0
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- added copper zone on B.Cu, net +12V
- removed copper zone on B.Cu, net /Motor 3/Motor Out A
- removed copper zone on F.Cu, net /Motor 3/Motor Out A
- removed copper zone on B.Cu, net /Motor 3/Motor Out B
- removed copper zone on F.Cu, net /Motor 3/Motor Out B
- removed copper zone on B.Cu, net /Motor 4/Motor Out A
- removed copper zone on F.Cu, net /Motor 4/Motor Out A
- removed copper zone on B.Cu, net /Motor 4/Motor Out B
- removed copper zone on F.Cu, net /Motor 4/Motor Out B
- removed copper zone on B.Cu, net Net-(C11-Pad1)
- removed copper zone on F.Cu, net Net-(C11-Pad1)
- removed copper zone on B.Cu, net Net-(C12-Pad1)
- removed copper zone on F.Cu, net Net-(C12-Pad1)
Other:
- board size 120 x 140 mm -> 150 x 180 mm
- board text added: "Project Inititum 2.0 PCB"
- board text added: "jlcjlcjlcjlc"
