File: elec/elec.kicad_sch (KiCad schematic)
At the start: 32 parts, among them J1 XT60-M, SW1 SW_SPST, SW2 SW_SPST, U1 TPS5430DDA, U2 TPS5430DDA, U3 4754

Commit message: completed?
Parts:
- removed SW1: SW_SPST, Connector_AMASS:AMASS_XT60-M_1x02_P7.20mm_Vertical, symbol Switch:SW_SPST
- removed TP1: TestPoint_2Pole, TestPoint:TestPoint_2Pads_Pitch2.54mm_Drill0.8mm, symbol Connector:TestPoint_2Pole
- added H1, H2, H3, H4: MountingHole, MountingHole:MountingHole_3.2mm_M3_Pad, symbol Mechanical:MountingHole
- added U9: 113991054, initium20:XiaoSeeedStudioEsp32, symbol XiaoSeeedStudioEsp32:113991054
- R5, R6: value R -> 10K
Connections:
- net +12V: now also J1.P (POS), TP2.2
- net +5V: now also U9.14 (VUSB)
- net GND: now also U9.13 (GND)
- net ESP32 RX: now reaches A1.20
- net ESP32 RX: now also U9.8 (RX_D7)
- net ESP32 TX: now reaches A1.21
- net ESP32 TX: now also U9.7 (TX_D6)
- net Motor 3 IN A: no longer names the net of A1.8
- net Motor 3 IN B: no longer names the net of A1.9
- net Motor 3 PWM: no longer names the net of A1.2
- net Motor 4 IN A: no longer names the net of A1.10
- net Motor 4 IN B: no longer names the net of A1.11
- net Motor 4 PWM: no longer names the net of A1.3
- no-connect marks 23 -> 37
Other:
- removed sheet Motor 3
- removed sheet Motor 4
- note added: "Mounting Holes"
- note removed: "10k"
- note removed: "???"
- note removed: "MORE BLANK SPACE"
- moved on the sheet: A1, R7, SW2, TP2, TP3, TP4, TP5, U4
